File: main_board/main_board.kicad_pcb (KiCad board)
At the start: 2 copper layers, 50.8 x 55.9 mm, 9 parts, among them J1 Conn_01x04_Socket, J2 Conn_01x04, J3 Conn_02x03_Odd_Even, J4 Conn_02x01, J5 Conn_02x02_Odd_Even, U1 Pico

Commit message: first commit
Parts:
- added J6: Conn_02x03_Odd_Even, Connector_PinHeader_2.54mm:PinHeader_2x03_P2.54mm_Vertical, F.Cu at (73.2, 48.8)
- added J7: Conn_02x01, Connector_PinHeader_2.54mm:PinHeader_2x01_P2.54mm_Vertical, F.Cu at (27.7, 42.7)
- added REF**: MountingHole_2.1mm, MountingHole:MountingHole_2.1mm, F.Cu at (29.7, 30.2)
- added SW1: SW_Push, Button_Switch_SMD:SW_Push_1P1T_NO_CK_PTS125Sx43PSMTR, B.Cu at (32.7, 63.8)
- J5: value Conn_02x02_Odd_Even -> Conn_02x01; footprint Connector_PinHeader_2.54mm:PinHeader_2x02_P2.54mm_Vertical -> Connector_PinHeader_2.54mm:PinHeader_2x01_P2.54mm_Vertical
- moved J5 111.0 mm to (27.7, 52.3)
- moved J4 84.1 mm to (27.7, 47.5), turned to 0 degrees
- moved REF** 79.9 mm to (29.7, 78.5)
- moved J1 76.4 mm to (36.1, 37.3)
- moved REF** 76.4 mm to (75.7, 61.0)
- moved REF** 76.4 mm to (79.2, 30.5)
- moved U1 76.4 mm to (55.4, 54.0)
- moved J2 76.4 mm to (73.4, 29.7)
- moved J3 76.4 mm to (74.2, 72.9)
Connections:
- J2 pad 2: /Ground -> GND
- J3 pad 1: /Ground -> GND
- J3 pad 2: /Ground -> GND
- J5 pad 1: /receiver1 -> /IR Out
- J5 pad 2: Net-(J5-Pin_2) -> GND
- U1 pad 13: unconnected-(U1-GND-Pad13) -> GND
- U1 pad 15: unconnected-(U1-GPIO11-Pad15) -> Net-(U1-GPIO11)
- U1 pad 18: unconnected-(U1-GND-Pad18) -> GND
- U1 pad 23: /Ground -> GND
- U1 pad 28: unconnected-(U1-GND-Pad28) -> GND
- U1 pad 3: unconnected-(U1-GND-Pad3) -> GND
- U1 pad 32: /receiver2 -> Net-(J6-Pin_1)
- U1 pad 33: unconnected-(U1-AGND-Pad33) -> GND
- U1 pad 34: /receiver1 -> Net-(J6-Pin_2)
- U1 pad 36: Net-(J5-Pin_2) -> Net-(J6-Pin_5)
- U1 pad 38: /Ground -> GND
Routing:
- net Net-(J6-Pin_5): track 0.00 -> 102.4 mm
- net GND: track 19.8 -> 100.7 mm
- net /Ground: track 42.7 -> 0.00 mm
- net Net-(U1-GPIO11): track 0.00 -> 37.2 mm
- net /IR Out: track 10.5 -> 29.8 mm
- net Net-(J5-Pin_2): track 15.5 -> 0.00 mm
- net /receiver1: track 10.8 -> 0.00 mm
- net /receiver2: track 10.1 -> 0.00 mm
- net Net-(J6-Pin_1): track 0.00 -> 9.83 mm
- net Net-(J6-Pin_2): track 0.00 -> 9.30 mm
- net /Light 1: track 17.1 -> 23.6 mm
- net /Light 2: track 13.5 -> 17.4 mm
- net /Light 4: track 16.6 -> 19.0 mm
Other:
- board size 50.8 x 55.9 mm -> 57.1 x 58.2 mm
- board text added: "3V3_EN"
- board text added: "GP18"
